File: Rb-controller-board.kicad_sch (KiCad schematic)
At the start: 44 parts, among them J1 Conn_02x05_Odd_Even, J2 Conn_Coaxial, J3 Screw_Terminal_01x03, J4 Conn_01x02, J5 Conn_Coaxial, J6 Conn_01x02, J7 Conn_01x02, U1 74AC04, U2 LM7805, U3 picDIV-10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

Commit message: Adjusted resistor values
RF termination resistor changed to 150 ohm to better match ribbon cable impedance.
Lower LED series resitors to 3k
Parts:
- R1, R13, R5: value 10k -> 3k
- R9: value 49.9 -> 150
Other:
- title: (none) -> Rubidium Interface board
